File: PCB/KiCad/GasWeighter.kicad_sch (KiCad schematic)
At the start: 14 parts, among them J1 3.7V Battery, J10 4Wire, J2 Solar Panel, J3 AA, J6 UL, J7 UR, J8 LL, J9 LR, P1 USB_C_Plug_USB2.0

Commit message: 3Cents USB
Parts:
- P1: footprint Library:USB C Molex -> Library:USB C Molex_1
Changed lines of the file:
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@@
       (effects (font (size 1.27 1.27)))
     )
-    (property "Footprint" "Library:USB C Molex" (at 38.1 99.06 0)
+    (property "Footprint" "Library:USB C Molex_1" (at 38.1 99.06 0)
       (effects (font (size 1.27 1.27)) hide)
     )
