File: PCB/KiCad/GasWeighter.kicad_pcb (KiCad board)
At the start: 2 copper layers, 74 x 50 mm, 84 parts, among them J1 3.7V Battery, J10 4Wire, J11 External Programming, J12 NTC, J2 Solar Panel, J3 AA, J6 UL, J7 UR, J8 LL, J9 LR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

Commit message: 3Cents USB
Parts:
- P1: footprint Library:USB C Molex -> Library:USB C Molex_1
- moved R14 5.74 mm to (126.9, 103.6), turned to 90 degrees
- moved R13 5.62 mm to (128.9, 103.6), turned to 90 degrees
- moved C6 2.90 mm to (127.5, 114.8)
- moved J1 2.06 mm to (114.0, 72.1)
- moved U4 1.38 mm to (127.5, 110.3)
- moved J12 0.20 mm to (123.2, 72.1)
Connections:
- SW1 pad 2: GND -> (no net)
- SW2 pad 2: GND -> (no net)
Routing:
- net GND: track 23.6 -> 14.1 mm, vias 17 -> 35
- net +3.3V: track 176.9 -> 169.6 mm
- net Net-(R6-Pad1): track 15.5 -> 10.5 mm
- net VCC: track 88.6 -> 92.4 mm
- net VBatt: track 19.6 -> 22.4 mm
- net Net-(R16-Pad1): track 10.6 -> 8.06 mm
- net /MCU/RX: track 56.3 -> 57.8 mm
- net /MCU/SDA: track 41.5 -> 42.8 mm
- net /MCU/SCL: track 42.1 -> 43.2 mm
- net Net-(JP7-A): track 2.43 -> 3.30 mm
Other:
- outline, holes or cut-outs redrawn
- board text added: "EN"
- board text removed: "Temp Sensors"

Commit message: Gerbers
Routing:
- net GND: vias 35 -> 36
Changed lines of the file:
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@@
     (pad "16" smd roundrect (at 2.5 -4.445 180) (size 2 0.6) (layers "F.Cu" "F.Paste" "F.Mask") (roundrect_rratio 0.25)
       (net 5 "+3.3V") (pinfunction "DVDD") (pintype "power_in"))
-    (model "${KICAD6_3DMODEL_DIR}/Package_SO.3dshapes/SOP-16_3.9x9.9mm_P1.27mm.wrl"
+    (model "${KICAD6_3DMODEL_DIR}/Package_SO.3dshapes/SOIC-16_3.9x9.9mm_P1.27mm.wrl"
       (offset (xyz 0 0 0))
       (scale (xyz 1 1 1))
@@
   (via (at 167.5 95) (size 0.5) (drill 0.3) (layers "F.Cu" "B.Cu") (free) (net 2))
   (via (at 112.4 80.95) (size 0.8) (drill 0.4) (layers "F.Cu" "B.Cu") (net 2))
+  (via (at 157.5 100) (size 0.5) (drill 0.3) (layers "F.Cu" "B.Cu") (free) (net 2))
   (via (at 175 92.5) (size 0.5) (drill 0.3) (layers "F.Cu" "B.Cu") (free) (net 2))
   (via (at 160 95) (size 0.5) (drill 0.3) (layers "F.Cu" "B.Cu") (free) (net 2))
